File: byteworker.sch (EAGLE design)
At the start: 59 parts, among them IC1 MCP1703, IC2 TJA1043, J2 AVRSPI-61.27, Q1 BSS138, Q2 BSS138, Q3 BSS138, Q4 AP2321GN-HF-3TR, Q5 BSS138, X1 16 MHz, X3 SUBD-H9

Commit message: v0.3.0: - swap subD connector for Male version. - center subD connector
Parts:
- removed X3: SUBD-H9, bytewerk-con:SUBD-H9
- added X2: SUBD-M_H9, bytewerk-con:SUBD-M_H9
Connections:
- net CANH: now also X27.F; no longer X37.F
- net CANL: now also X22.F; no longer X32.F
- net GND: now also X23.F; no longer X33.F
- net VIN_BUS: now also X29.F; no longer X39.F
Changed lines of the file:
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@@
 <part name="JP2" library="pinhead" deviceset="PINHD-1X6" device=""/>
 <part name="Q4" library="bytewerk-transistor" deviceset="AP2321GN-HF-3TR" device=""/>
-<part name="X3" library="bytewerk-con" deviceset="SUBD" device="-H9"/>
 <part name="D4" library="bytewerk-diode" deviceset="ZENER" device="_PTVS18VP1UP" value="16V"/>
 <part name="U$3" library="bytewerk-symbol" deviceset="GND" device=""/>
+<part name="X2" library="bytewerk-con" deviceset="SUBD" device="-M_H9"/>
 </parts>
 <sheets>
@@
 <description>Connector</description>
 <plain>
-<text x="137.16" y="137.16" size="1.778" layer="98" align="center-right">7V to 16V</text>
+<text x="185.42" y="137.16" size="1.778" layer="98" align="center-right">7V to 16V</text>
 <text x="190.5" y="99.06" size="1.778" layer="98" rot="R180" align="center-right">7V to 16V</text>
 <text x="71.12" y="142.24" size="1.778" layer="98" align="center-left">max 50mA</text>
@@
 <instance part="JP3" gate="A" x="165.1" y="109.22" rot="R180"/>
 <instance part="JP2" gate="A" x="149.86" y="93.98" rot="R90"/>
-<instance part="X3" gate="1" x="157.48" y="157.48"/>
-<instance part="X3" gate="2" x="157.48" y="154.94"/>
-<instance part="X3" gate="3" x="157.48" y="152.4"/>
-<instance part="X3" gate="4" x="157.48" y="149.86"/>
-<instance part="X3" gate="5" x="157.48" y="147.32"/>
-<instance part="X3" gate="6" x="157.48" y="144.78"/>
-<instance part="X3" gate="7" x="157.48" y="142.24"/>
-<instance part="X3" gate="8" x="157.48" y="139.7"/>
-<instance part="X3" gate="9" x="157.48" y="137.16"/>
+<instance part="X2" gate="1" x="205.74" y="157.48"/>
+<instance part="X2" gate="2" x="205.74" y="154.94"/>
+<instance part="X2" gate="3" x="205.74" y="152.4"/>
+<instance part="X2" gate="4" x="205.74" y="149.86"/>
+<instance part="X2" gate="5" x="205.74" y="147.32"/>
+<instance part="X2" gate="6" x="205.74" y="144.78"/>
+<instance part="X2" gate="7" x="205.74" y="142.24"/>
+<instance part="X2" gate="8" x="205.74" y="139.7"/>
+<instance part="X2" gate="9" x="205.74" y="137.16"/>
 </instances>
 <busses>
@@
 <net name="VIN_BUS" class="0">
 <segment>
-<pinref part="X3" gate="9" pin="F"/>
-<wire x1="154.94" y1="137.16" x2="152.4" y2="137.16" width="0.1524" layer="91"/>
-<label x="152.4" y="137.16" size="1.27" layer="95" rot="MR0" xref="yes"/>
+<pinref part="X2" gate="9" pin="F"/>
+<wire x1="200.66" y1="137.16" x2="203.2" y2="137.16" width="0.1524" layer="91"/>
+<label x="200.66" y="137.16" size="1.27" layer="95" rot="MR0" xref="yes"/>
 </segment>
 </net>
@@
 </segment>
 <segment>
-<pinref part="X3" gate="3" pin="F"/>
-<wire x1="154.94" y1="152.4" x2="152.4" y2="152.4" width="0.1524" layer="91"/>
-<label x="152.4" y="152.4" size="1.27" layer="95" rot="MR0" xref="yes"/>
+<pinref part="X2" gate="3" pin="F"/>
+<wire x1="203.2" y1="152.4" x2="200.66" y2="152.4" width="0.1524" layer="91"/>
+<label x="200.66" y="152.4" size="1.27" layer="95" rot="MR0" xref="yes"/>
 </segment>
 </net>
@@
 </segment>
 <segment>
-<pinref part="X3" gate="7" pin="F"/>
-<wire x1="154.94" y1="142.24" x2="152.4" y2="142.24" width="0.1524" layer="91"/>
-<label x="152.4" y="142.24" size="1.27" layer="95" rot="MR0" xref="yes"/>
+<pinref part="X2" gate="7" pin="F"/>
+<wire x1="203.2" y1="142.24" x2="200.66" y2="142.24" width="0.1524" layer="91"/>
+<label x="200.66" y="142.24" size="1.27" layer="95" rot="MR0" xref="yes"/>
 </segment>
 </net>
@@
 </segment>
 <segment>
-<pinref part="X3" gate="2" pin="F"/>
-<wire x1="154.94" y1="154.94" x2="152.4" y2="154.94" width="0.1524" layer="91"/>
-<label x="152.4" y="154.94" size="1.27" layer="95" rot="MR0" xref="yes"/>
+<pinref part="X2" gate="2" pin="F"/>
+<wire x1="203.2" y1="154.94" x2="200.66" y2="154.94" width="0.1524" layer="91"/>
+<label x="200.66" y="154.94" size="1.27" layer="95" rot="MR0" xref="yes"/>
 </segment>
 </net>
