File: byteworker.sch (EAGLE design)
At the start: 59 parts, among them IC1 MCP1703, IC2 TJA1043, J2 AVRSPI-61.27, Q1 BSS138, Q2 BSS138, Q3 BSS138, Q4 AP2321GN-HF-3TR, Q5 BSS138, X1 16 MHz, X2 SUBD-M_H9

Commit message: v0.4.0: - 500 mA +5V voltage regulator with larger package and input voltage - female sub-d connector - thicker power traces - removed 1 test-led
Parts:
- removed IC1: MCP1703, bytewerk-vreg:MCP1703
- removed LED1: green, bytewerk-led:LED0603
- removed R21: 1k, bytewerk-passive:R0603
- added IC3: UA78M05IDCY, bytewerk-vreg:UA78M05IDCY
- C2: value 1u/25V -> 100n; device bytewerk-rcl:C1206 -> bytewerk-passive:C0603
- C3: value 1u/10V -> 330n; device bytewerk-rcl:C1206 -> bytewerk-passive:C0603
- R7: value n.b.[1k] -> 1k
Connections:
- removed net N$7: LED1.A, R21.2
- removed net TESTLED1: R21.1, UC1PORTC.(AMP1+/ACMP3/ADC9)PC5
- net +5V: now also C2.1, IC3.+5V; no longer C3.1, IC1.VCC
- net GND: now also IC3.GND; no longer IC1.GND, LED1.C
- net VOUT_SW: now also C3.1, IC3.VIN; no longer C2.1, IC1.VIN
Other:
- note added: "7V to 35V"
- note added: "max 250mA"
- note removed: "7V to 16V"
- note removed: "max 150 mA"
- note removed: "max 50mA"
- moved on the sheet: C2, C3
Changed lines of the file:
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@@
 <parts>
 <part name="UC1" library="bytewerk-uc" deviceset="ATMEGA16M1" device=""/>
-<part name="IC1" library="bytewerk-vreg" deviceset="MCP1703" device="">
-<attribute name="OC_MOUSER" value="579-mcp1703T-5002ECB"/>
-</part>
-<part name="C2" library="bytewerk-rcl" deviceset="C" device="1206" value="1u/25V"/>
 <part name="GND1" library="supply1" deviceset="GND" device=""/>
 <part name="GND3" library="supply1" deviceset="GND" device=""/>
@@
 <part name="C7" library="bytewerk-passive" deviceset="C" device="0603" value="100n"/>
 <part name="GND11" library="supply1" deviceset="GND" device=""/>
-<part name="C3" library="bytewerk-rcl" deviceset="C" device="1206" value="1u/10V"/>
 <part name="GND2" library="supply1" deviceset="GND" device=""/>
 <part name="Q5" library="bytewerk-fet" deviceset="BSS138" device=""/>
@@
 <part name="R11" library="bytewerk-rcl" deviceset="R" device="0603" value="dnp"/>
 <part name="P+3" library="supply1" deviceset="+5V" device=""/>
-<part name="R21" library="bytewerk-passive" deviceset="R" device="0603" value="1k"/>
 <part name="R22" library="bytewerk-passive" deviceset="R" device="0603" value="1k"/>
 <part name="J2" library="bytewerk-con" deviceset="AVRSPI-6" device="1.27"/>
 <part name="JP1" library="pinhead" deviceset="PINHD-1X10" device=""/>
 <part name="JP3" library="pinhead" deviceset="PINHD-1X10" device=""/>
-<part name="LED1" library="bytewerk-led" deviceset="LED0603" device="" value="green"/>
 <part name="U$1" library="bytewerk-symbol" deviceset="GND" device=""/>
 <part name="LED2" library="bytewerk-led" deviceset="LED0603" device="" value="blue"/>
@@
 <part name="D6" library="bytewerk-passive" deviceset="SCHOTTKY" device="323"/>
 <part name="LED3" library="bytewerk-led" deviceset="LED0603" device="" value="red"/>
-<part name="R7" library="bytewerk-passive" deviceset="R" device="0603" value="n.b.[1k]"/>
+<part name="R7" library="bytewerk-passive" deviceset="R" device="0603" value="1k"/>
 <part name="GND20" library="supply1" deviceset="GND" device=""/>
 <part name="JP2" library="pinhead" deviceset="PINHD-1X6" device=""/>
@@
 <part name="U$3" library="bytewerk-symbol" deviceset="GND" device=""/>
 <part name="X2" library="bytewerk-con" deviceset="SUBD" device="-M_H9"/>
+<part name="IC3" library="bytewerk-vreg" deviceset="UA78M05IDCY" device=""/>
+<part name="C3" library="bytewerk-passive" deviceset="C" device="0603" value="330n"/>
+<part name="C2" library="bytewerk-passive" deviceset="C" device="0603" value="100n"/>
 </parts>
 <sheets>
@@
 <description>Connector</description>
 <plain>
-<text x="185.42" y="137.16" size="1.778" layer="98" align="center-right">7V to 16V</text>
-<text x="190.5" y="99.06" size="1.778" layer="98" rot="R180" align="center-right">7V to 16V</text>
-<text x="71.12" y="142.24" size="1.778" layer="98" align="center-left">max 50mA</text>
-<text x="185.42" y="121.92" size="1.778" layer="98" rot="R180" align="center-right">max 50mA</text>
+<text x="185.42" y="137.16" size="1.778" layer="98" align="center-right">7V to 35V</text>
+<text x="190.5" y="99.06" size="1.778" layer="98" rot="R180" align="center-right">7V to 35V</text>
+<text x="71.12" y="142.24" size="1.778" layer="98" align="center-left">max 250mA</text>
+<text x="185.42" y="121.92" size="1.778" layer="98" rot="R180" align="center-right">max 250mA</text>
 </plain>
 <instances>
@@
 <description>Power &amp; CAN</description>
 <plain>
-<text x="231.14" y="149.86" size="1.778" layer="98" align="top-left">max 150 mA</text>
+<text x="231.14" y="149.86" size="1.778" layer="98" align="top-left">max 250mA</text>
 </plain>
 <instances>
 <instance part="FRAME3" gate="G$1" x="0" y="0"/>
-<instance part="IC1" gate="G$1" x="213.36" y="137.16"/>
-<instance part="C2" gate="G$1" x="193.04" y="124.46" rot="R270"/>
 <instance part="GND1" gate="1" x="193.04" y="109.22"/>
 <instance part="GND3" gate="1" x="213.36" y="109.22"/>
-<instance part="C3" gate="G$1" x="226.06" y="124.46" rot="R270"/>
 <instance part="GND2" gate="1" x="226.06" y="109.22"/>
 <instance part="Q5" gate="G$1" x="180.34" y="121.92"/>
@@
 <instance part="D4" gate="G$1" x="162.56" y="154.94" rot="R180"/>
 <instance part="U$3" gate="G$1" x="170.18" y="149.86"/>
+<instance part="IC3" gate="G$1" x="213.36" y="137.16"/>
+<instance part="C3" gate="G$1" x="193.04" y="124.46" rot="R270"/>
+<instance part="C2" gate="G$1" x="226.06" y="124.46" rot="R270"/>
 </instances>
 <busses>
@@
 <net name="GND" class="0">
 <segment>
-<pinref part="C2" gate="G$1" pin="2"/>
 <wire x1="193.04" y1="111.76" x2="193.04" y2="121.92" width="0.1524" layer="91"/>
 <pinref part="GND1" gate="1" pin="GND"/>
-</segment>
-<segment>
-<pinref part="IC1" gate="G$1" pin="GND"/>
+<pinref part="C3" gate="G$1" pin="2"/>
+</segment>
+<segment>
 <pinref part="GND3" gate="1" pin="GND"/>
 <wire x1="213.36" y1="111.76" x2="213.36" y2="132.08" width="0.1524" layer="91"/>
-</segment>
-<segment>
-<pinref part="C3" gate="G$1" pin="2"/>
+<pinref part="IC3" gate="G$1" pin="GND"/>
+</segment>
+<segment>
 <pinref part="GND2" gate="1" pin="GND"/>
 <wire x1="226.06" y1="121.92" x2="226.06" y2="111.76" width="0.1524" layer="91"/>
+<pinref part="C2" gate="G$1" pin="2"/>
 </segment>
 <segment>
@@
 <net name="+5V" class="0">
 <segment>
-<pinref part="IC1" gate="G$1" pin="VCC"/>
 <wire x1="223.52" y1="139.7" x2="226.06" y2="139.7" width="0.1524" layer="91"/>
 <wire x1="226.06" y1="139.7" x2="226.06" y2="147.32" width="0.1524" layer="91"/>
 <label x="231.14" y="152.4" size="1.778" layer="95" xref="yes"/>
-<pinref part="C3" gate="G$1" pin="1"/>
 <wire x1="226.06" y1="147.32" x2="226.06" y2="152.4" width="0.1524" layer="91"/>
 <wire x1="226.06" y1="129.54" x2="226.06" y2="139.7" width="0.1524" layer="91"/>
@@
 <pinref part="D6" gate="G$1" pin="A"/>
 <wire x1="218.44" y1="147.32" x2="226.06" y2="147.32" width="0.1524" layer="91"/>
+<pinref part="IC3" gate="G$1" pin="+5V"/>
+<pinref part="C2" gate="G$1" pin="1"/>
 </segment>
 <segment>
@@
 <net name="VOUT_SW" class="0">
 <segment>
-<pinref part="IC1" gate="G$1" pin="VIN"/>
 <wire x1="190.5" y1="139.7" x2="193.04" y2="139.7" width="0.1524" layer="91"/>
-<pinref part="C2" gate="G$1" pin="1"/>
 <wire x1="193.04" y1="139.7" x2="200.66" y2="139.7" width="0.1524" layer="91"/>
 <wire x1="200.66" y1="139.7" x2="203.2" y2="139.7" width="0.1524" layer="91"/>
@@
 <junction x="200.66" y="139.7"/>
 <pinref part="Q4" gate="G$1" pin="D"/>
+<pinref part="IC3" gate="G$1" pin="VIN"/>
+<pinref part="C3" gate="G$1" pin="1"/>
 </segment>
 </net>
@@
 <instance part="R11" gate="G$1" x="129.54" y="149.86" rot="MR180"/>
 <instance part="P+3" gate="1" x="144.78" y="144.78" rot="MR90"/>
-<instance part="R21" gate="G$1" x="119.38" y="53.34" rot="MR180"/>
 <instance part="R22" gate="G$1" x="119.38" y="48.26" rot="MR180"/>
-<instance part="LED1" gate="G$1" x="129.54" y="53.34"/>
 <instance part="U$1" gate="G$1" x="142.24" y="43.18"/>
 <instance part="LED2" gate="G$1" x="129.54" y="48.26"/>
@@
 </segment>
 <segment>
-<pinref part="LED1" gate="G$1" pin="C"/>
-<wire x1="132.08" y1="53.34" x2="142.24" y2="53.34" width="0.1524" layer="91"/>
 <pinref part="U$1" gate="G$1" pin="GND"/>
-<wire x1="142.24" y1="53.34" x2="142.24" y2="48.26" width="0.1524" layer="91"/>
 <pinref part="LED2" gate="G$1" pin="C"/>
 <wire x1="142.24" y1="48.26" x2="142.24" y2="45.72" width="0.1524" layer="91"/>
 <wire x1="132.08" y1="48.26" x2="142.24" y2="48.26" width="0.1524" layer="91"/>
-<junction x="142.24" y="48.26"/>
 </segment>
 </net>
@@
 </segment>
 </net>
-<net name="TESTLED1" class="0">
-<segment>
-<pinref part="UC1" gate="PORTC" pin="(AMP1+/ACMP3/ADC9)PC5"/>
-<pinref part="R21" gate="G$1" pin="1"/>
-<wire x1="114.3" y1="53.34" x2="111.76" y2="53.34" width="0.1524" layer="91"/>
-<wire x1="111.76" y1="53.34" x2="111.76" y2="50.8" width="0.1524" layer="91"/>
-<wire x1="111.76" y1="50.8" x2="58.42" y2="50.8" width="0.1524" layer="91"/>
-</segment>
-</net>
 <net name="TESTLED2" class="0">
 <segment>
@@
 </segment>
 </net>
-<net name="N$7" class="0">
-<segment>
-<pinref part="LED1" gate="G$1" pin="A"/>
-<pinref part="R21" gate="G$1" pin="2"/>
-<wire x1="127" y1="53.34" x2="124.46" y2="53.34" width="0.1524" layer="91"/>
-</segment>
-</net>

Commit message: v4.1: add 2nd test LED
Parts:
- added LED1: red, bytewerk-led:LED0603
- added R21: 1k, bytewerk-passive:R0603
Connections:
- new net N$7: LED1.A, UC1PORTC.(AMP1+/ACMP3/ADC9)PC5
- new net N$9: LED1.C, R21.1
- net GND: now also R21.2
Changed lines of the file:
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@@
 <part name="C3" library="bytewerk-passive" deviceset="C" device="0603" value="330n"/>
 <part name="C2" library="bytewerk-passive" deviceset="C" device="0603" value="100n"/>
+<part name="R21" library="bytewerk-passive" deviceset="R" device="0603" value="1k"/>
+<part name="LED1" library="bytewerk-led" deviceset="LED0603" device="" value="red"/>
 </parts>
 <sheets>
@@
 <instance part="LED2" gate="G$1" x="129.54" y="48.26"/>
 <instance part="C10" gate="G$1" x="180.34" y="81.28" rot="R180"/>
+<instance part="R21" gate="G$1" x="132.08" y="53.34" rot="MR180"/>
+<instance part="LED1" gate="G$1" x="119.38" y="53.34"/>
 </instances>
 <busses>
@@
 <wire x1="142.24" y1="48.26" x2="142.24" y2="45.72" width="0.1524" layer="91"/>
 <wire x1="132.08" y1="48.26" x2="142.24" y2="48.26" width="0.1524" layer="91"/>
+<wire x1="142.24" y1="53.34" x2="142.24" y2="48.26" width="0.1524" layer="91"/>
+<junction x="142.24" y="48.26"/>
+<pinref part="R21" gate="G$1" pin="2"/>
+<wire x1="137.16" y1="53.34" x2="142.24" y2="53.34" width="0.1524" layer="91"/>
 </segment>
 </net>
@@
 </segment>
 </net>
+<net name="N$7" class="0">
+<segment>
+<pinref part="UC1" gate="PORTC" pin="(AMP1+/ACMP3/ADC9)PC5"/>
+<wire x1="58.42" y1="50.8" x2="73.66" y2="50.8" width="0.1524" layer="91"/>
+<wire x1="111.76" y1="53.34" x2="111.76" y2="50.8" width="0.1524" layer="91"/>
+<wire x1="111.76" y1="50.8" x2="73.66" y2="50.8" width="0.1524" layer="91"/>
+<pinref part="LED1" gate="G$1" pin="A"/>
+<wire x1="111.76" y1="53.34" x2="116.84" y2="53.34" width="0.1524" layer="91"/>
+</segment>
+</net>
+<net name="N$9" class="0">
+<segment>
+<pinref part="LED1" gate="G$1" pin="C"/>
+<pinref part="R21" gate="G$1" pin="1"/>
+<wire x1="121.92" y1="53.34" x2="127" y2="53.34" width="0.1524" layer="91"/>
+</segment>
+</net>
